File: board/cartteFille/button.kicad_sch (KiCad schematic)
At the start: 13 parts, among them U27-8 SN74LVC2G14DBVTG4

Commit message: resistor tab adding
on rajoute une table de résistance pour le changement facile de boutons
Parts:
- renumbered C271 to C211, C281 to C221, D27 to D21, D28 to D22, R271 to R211, R272 to R212, R273 to R213, R281 to R221, R282 to R222, R283 to R223, S27 to S21, S28 to S22, U27-8 to U21-2
Other:
- note added: "1"
- note added: "1.5k"
- note added: "1.8"
- note added: "1.8k"
- note added: "10"
- note added: "120"
- note added: "150"
- note added: "2"
- note added: "2.1"
- note added: "20"
- note added: "3.3"
- note added: "3.3k"
- note added: "3.9"
- note added: "5"
- note added: "68"
- note added: "820"
- note added: "Alim 3.3 or 5 [V]"
- note added: "All resistors consume less than 125mW so power rating 1/8 pacage ex: 1206 footprint determination!"
- note added: "Led If [mA]"
- note added: "Led Vf [V]"
- note added: "Led color"
- note added: "R213&R223 Value given a LED"
- note added: "R2?3 Value [Ohm]"
- note added: "X"
- note added: "blue"
- note added: "orange"
- note added: "pure green"
- note added: "super red"
- note added: "yellow"

Commit message: end of the day
Parts:
- renumbered C211 to C271, C221 to C281, D21 to D27, D22 to D28, R211 to R271, R212 to R272, R213 to R273, R221 to R281, R222 to R282, R223 to R283, S21 to S27, S22 to S28, U21-2 to U27-8
Other:
- note added: "2-Current Regulator 20mA"
- note added: "RC Filter fc ~160Hz"
- note removed: "2-Current Regulator"
- note removed: "RC Filter"
- moved on the sheet: D27, D28
