File: board/cartteFille/cartteFille.kicad_sch (KiCad schematic)
At the start: 13 parts, among them U1 LM358, U20 MCP23018-E/SS

Commit message: litle change
Parts:
- renumbered R12 to R11, R11 to R12
Other:
- note added: "RC Filter fc ~160Hz"
- note removed: "RC Filter"
Changed lines of the file:
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@@
     (effects (font (size 1 1)) (justify left bottom))
   )
-  (text "RC Filter" (at 243.459 54.102 0)
+  (text "RC Filter\nfc ~160Hz" (at 243.84 55.88 0)
     (effects (font (size 1.5 1.5) (thickness 0.3) bold italic) (justify left bottom))
   )
@@
   (symbol (lib_id "Device:R") (at 202.184 56.642 90) (unit 1)
     (in_bom yes) (on_board yes) (fields_autoplaced)
-    (property "Reference" "R11" (id 0) (at 202.184 50.292 90))
-    (property "Value" "150Ohm" (id 1) (at 202.184 52.832 90))
+    (property "Reference" "R12" (id 0) (at 202.184 50.8 90))
+    (property "Value" "150Ohm" (id 1) (at 202.184 53.34 90))
     (property "Footprint" "Resistor_SMD:R_0603_1608Metric" (id 2) (at 202.184 58.42 90)
       (effects (font (size 1.27 1.27)) hide)
@@
   (symbol (lib_id "Device:R") (at 235.839 59.182 90) (unit 1)
     (in_bom yes) (on_board yes) (fields_autoplaced)
-    (property "Reference" "R12" (id 0) (at 235.839 52.832 90))
-    (property "Value" "10KOhm" (id 1) (at 235.839 55.372 90))
+    (property "Reference" "R11" (id 0) (at 235.839 53.34 90))
+    (property "Value" "10KOhm" (id 1) (at 235.839 55.88 90))
     (property "Footprint" "Resistor_SMD:R_0603_1608Metric" (id 2) (at 235.839 60.96 90)
       (effects (font (size 1.27 1.27)) hide)
@@
       (reference "EXT2") (unit 1) (value "NS(HN1x10)") (footprint "connecteur:HN1x10")
     )
+    (path "/abe955ed-02be-49ba-b797-c5f3c376f3ac"
+      (reference "R11") (unit 1) (value "10KOhm") (footprint "Resistor_SMD:R_0603_1608Metric")
+    )
     (path "/1aa5a763-bcca-4c6a-a02c-fa18c5b433a2"
-      (reference "R11") (unit 1) (value "150Ohm") (footprint "Resistor_SMD:R_0603_1608Metric")
-    )
-    (path "/abe955ed-02be-49ba-b797-c5f3c376f3ac"
-      (reference "R12") (unit 1) (value "10KOhm") (footprint "Resistor_SMD:R_0603_1608Metric")
+      (reference "R12") (unit 1) (value "150Ohm") (footprint "Resistor_SMD:R_0603_1608Metric")
     )
     (path "/a1b97586-5ccb-4d4b-808f-ce5452376c86"
